File: peregrine-pcb/peregrine.kicad_pcb (KiCad board)
At the start: 4 copper layers, 65 x 35 mm, 48 parts, among them J1 MEM2061-01-188-00-A_REVA, J3 Conn_01x02_Pin, J4 USB4105-GF-A, Q2 FSB560A, U1 RP2040, U2 W25Q32JVZP, U3 AP63203WU, U4 BMP581, U5 ISM330DLCTR, Y1 ECS-120-20-33-AEL-TR

Commit message: first pass for pcb
Parts:
- removed J3: Conn_01x02_Pin, Connector_PinHeader_1.00mm:PinHeader_1x02_P1.00mm_Vertical
- added C18: 100nF, Capacitor_SMD:C_0603_1608Metric, F.Cu at (128.2, 104.5)
- added D3: 1N4148WT, Diode_SMD:D_SOD-523, F.Cu at (142.8, 123.5)
- added D4: 1N4148WT, Diode_SMD:D_SOD-523, F.Cu at (142.8, 122.0)
- added D5: LSM115JE3/TR13, LSM115JE3:DO-214BA_MCH, F.Cu at (111.5, 116.0)
- added D6: LSM115JE3/TR13, LSM115JE3:DO-214BA_MCH, F.Cu at (116.0, 116.0)
- added J2: Screw_Terminal_01x04, YO0421500000G:CONN4_500000G_AMP, F.Cu at (104.0, 112.7)
- added J5: Screw_Terminal_01x04, YO0421500000G:CONN4_500000G_AMP, F.Cu at (161.0, 123.6)
- added J6: USB_C_Receptacle_USB2.0_16P, Connector_USB:USB_C_Receptacle_GCT_USB4105-xx-A_16P_TopMnt_Horizontal, F.Cu at (132.5, 131.5)
- added R16: 10k, Resistor_SMD:R_0603_1608Metric, F.Cu at (147.1, 123.2)
- added R17: 10k, Resistor_SMD:R_0603_1608Metric, F.Cu at (147.2, 121.2)
- added R18: 220, Resistor_SMD:R_0603_1608Metric, F.Cu at (147.2, 119.8)
- added R19: 10k, Resistor_SMD:R_0603_1608Metric, F.Cu at (147.2, 114.0)
- added R20: 10k, Resistor_SMD:R_0603_1608Metric, F.Cu at (147.2, 116.0)
- added R21: 66.5, Resistor_SMD:R_0603_1608Metric, F.Cu at (140.1, 122.0)
- added R22: 66.5, Resistor_SMD:R_0603_1608Metric, F.Cu at (140.1, 123.5)
- added R23: 220, Resistor_SMD:R_0603_1608Metric, F.Cu at (147.2, 112.5)
- added U6: VN5E160STR-E, VN5E160STR:SOIC127P600X175-8N, F.Cu at (152.8, 121.8)
- added U7: VN5E160STR-E, VN5E160STR:SOIC127P600X175-8N, F.Cu at (152.8, 114.5)
- J4: value USB4105-GF-A -> Conn_01x03_Pin; footprint Connector_USB:USB_C_Receptacle_GCT_USB4105-xx-A_16P_TopMnt_Horizontal -> Connector_PinHeader_2.54mm:PinHeader_1x03_P2.54mm_Vertical
- R8, R9: value R -> 10k
- moved R7 89.2 mm to (155.2, 132.6), turned to -90 degrees
- moved C13 87.5 mm to (158.5, 126.8)
- moved D2 87.3 mm to (156.8, 132.6), turned to -90 degrees
- moved C14 87.1 mm to (158.5, 128.3)
- moved R6 85.3 mm to (151.2, 132.6), turned to -90 degrees
- moved R1 78.7 mm to (104.8, 127.5)
- moved C17 76.6 mm to (148.2, 133.0), turned to -90 degrees
- moved C15 76.1 mm to (154.3, 107.5), turned to 180 degrees
- moved C16 75.9 mm to (154.3, 109.0)
- moved D1 72.1 mm to (152.7, 132.6), turned to -90 degrees
- moved U5 68.6 mm to (150.8, 108.5), turned to 90 degrees
- moved R10 61.6 mm to (144.0, 105.5), turned to -90 degrees
- moved R11 59.7 mm to (142.5, 105.5), turned to -90 degrees
- moved R8 56.6 mm to (136.4, 109.0), turned to 180 degrees
- moved R9 56.2 mm to (136.4, 110.5), turned to 180 degrees
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Connections:
- R2 pad 1: Net-(J4-CC1) -> Net-(J6-CC1)
- R3 pad 1: Net-(J4-CC2) -> Net-(J6-CC2)
- R4 pad 1: Net-(J4-D--PadA7) -> Net-(J6-D--PadA7)
- R5 pad 1: Net-(J4-D+-PadA6) -> Net-(J6-D+-PadA6)
- U1 pad 13: unconnected-(U1-GPIO10-Pad13) -> MAIN_FIRE
- U1 pad 14: unconnected-(U1-GPIO11-Pad14) -> DROGUE_FIRE
- U1 pad 24: Net-(J3-Pin_1) -> Net-(J4-Pin_1)
- U1 pad 25: Net-(J3-Pin_2) -> Net-(J4-Pin_3)
Routing:
- net SDA: track 0.00 -> 56.2 mm, vias 0 -> 4
- net Net-(J4-Pin_3): track 0.00 -> 55.4 mm, vias 0 -> 1
- net SCL: track 0.00 -> 54.6 mm, vias 0 -> 4
- net Net-(J4-Pin_1): track 0.00 -> 47.3 mm, vias 0 -> 1
- net MAIN_FIRE: track 0.00 -> 46.6 mm, vias 0 -> 5
- net GND: track 37.2 -> 83.7 mm, vias 8 -> 37
- net DROGUE_FIRE: track 0.00 -> 40.0 mm, vias 0 -> 4
- net LED_1: track 0.00 -> 35.7 mm, vias 0 -> 2
- net RUN: track 0.00 -> 30.8 mm, vias 0 -> 1
- net VBUS: track 6.89 -> 35.8 mm, vias 0 -> 4
- net SD_DETECT: track 0.00 -> 27.3 mm, vias 0 -> 2
- net QSPI_SS: track 10.1 -> 36.9 mm, vias 0 -> 2
- net +3V3: track 43.2 -> 67.9 mm, vias 17 -> 31
- net SD_CS: track 0.00 -> 23.5 mm, vias 0 -> 2
- net BUZZER: track 0.00 -> 19.4 mm, vias 0 -> 2
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- added copper zone on F.Cu, net GND
- added copper zone on F.Cu, net Net-(D3-K)
- added copper zone on F.Cu, net Net-(D4-K)
- added copper zone on F.Cu, net VCCB
- added copper zone on F.Cu, net V_BATT
- removed copper zone on B.Cu, net VCCB
Other:
- outline, holes or cut-outs redrawn
- board text added: "JLCJLCJLCJLC"
- board text added: "Peregrine v0.1"
- board text added: "SWCLK GND SWD"
- board text added: "Tim Gibson"
