File: peregrine-pcb/peregrine.kicad_sch (KiCad schematic)
At the start: 49 parts, among them J1 MEM2061-01-188-00-A_REVA, J2 Screw_Terminal_01x04, J3 Conn_01x02_Pin, J4 USB4105-GF-A, Q2 FSB560A, U1 RP2040, U2 W25Q32JVZP, U3 AP63203WU, U4 BMP581, U5 ISM330DLCTR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

Commit message: first pass for pcb
Parts:
- removed J3: Conn_01x02_Pin, Connector_PinHeader_1.00mm:PinHeader_1x02_P1.00mm_Vertical, symbol Connector:Conn_01x02_Pin
- removed J4: USB4105-GF-A, Connector_USB:USB_C_Receptacle_GCT_USB4105-xx-A_16P_TopMnt_Horizontal, symbol Connector:USB_C_Receptacle
- added C18: 100nF, Capacitor_SMD:C_0603_1608Metric, symbol Device:C
- added D3, D4: 1N4148WT, Diode_SMD:D_SOD-523, symbol Diode:1N4148WT
- added D5, D6: LSM115JE3/TR13, LSM115JE3:DO-214BA_MCH, symbol Device:D
- added J4: Conn_01x03_Pin, Connector_PinHeader_2.54mm:PinHeader_1x03_P2.54mm_Vertical, symbol Connector:Conn_01x03_Pin
- added J5: Screw_Terminal_01x04, YO0421500000G:CONN4_500000G_AMP, symbol Connector:Screw_Terminal_01x04
- added J6: USB_C_Receptacle_USB2.0_16P, Connector_USB:USB_C_Receptacle_GCT_USB4105-xx-A_16P_TopMnt_Horizontal, symbol Connector:USB_C_Receptacle_USB2.0_16P
- added R16, R17, R19, R20: 10k, Resistor_SMD:R_0603_1608Metric, symbol Device:R
- added R18, R23: 220, Resistor_SMD:R_0603_1608Metric, symbol Device:R
- added R21, R22: 66.5, Resistor_SMD:R_0603_1608Metric, symbol Device:R
- added U6, U7: VN5E160STR-E, VN5E160STR:SOIC127P600X175-8N, symbol VN5E160STR-E:VN5E160STR-E
- J2: footprint (none) -> YO0421500000G:CONN4_500000G_AMP
- R8, R9: value R -> 10k
Connections:
- net +3V3: now also C18.1, R16.1, R20.1
- net DROGUE_CONT: now also R21.1
- net GND: now also C18.2, J4.2 (Pin_2), J5.2 (Pin_2), J5.4 (Pin_4), J6.A1 (GND), J6.A12 (GND), J6.B1 (GND), J6.B12 (GND), R17.2, R18.2, R19.2, R23.2
- net MAIN_CONT: now also R22.1
- net VBUS: now also D6.2 (A), J6.A4 (VBUS), J6.A9 (VBUS), J6.B4 (VBUS), J6.B9 (VBUS)
- net VCCB: now also D5.1 (K), D6.1 (K); no longer J2.1 (Pin_1)
- net at R2.1: now also J6.A5 (CC1)
- net at R3.1: now also J6.B5 (CC2)
- net at R4.1: now also J6.A7 (D-), J6.B7 (D-)
- net MAIN_FIRE: now reaches U1.13 (GPIO10)
- net MAIN_FIRE: now also R17.1, U6.2 (INPUT)
- net DROGUE_FIRE: now reaches U1.14 (GPIO11)
- net DROGUE_FIRE: now also R19.1, U7.2 (INPUT)
- net at U1.24 (SWCLK): now also J4.1 (Pin_1)
- net at U1.25 (SWD): now also J4.3 (Pin_3)
- net at R5.1: now also J6.A6 (D+), J6.B6 (D+)
- new net: D3.1 (K), J5.1 (Pin_1), U6.6 (OUTPUT), U6.7 (OUTPUT__1)
- new net: D3.2 (A), R22.2
- new net: R20.2, U7.4 (STAT_DIS)
- new net: D4.2 (A), R21.2
- new net: R23.1, U7.1 (GND)
- new net: D4.1 (K), J5.3 (Pin_3), U7.6 (OUTPUT), U7.7 (OUTPUT__1)
- new net: R18.1, U6.1 (GND)
- new net: R16.2, U6.4 (STAT_DIS)
- new net V_BATT: D5.2 (A), J2.1 (Pin_1), U6.5 (VCC), U6.8 (VCC__1), U7.5 (VCC), U7.8 (VCC__1)
- no-connect marks 18 -> 28
Other:
- moved on the sheet: C13, C14, C15, C16, C3, C4, C5, C6, J2, R1, R10, R11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
